File: RSHP-CB.kicad_pcb (KiCad board)
At the start: 2 copper layers, 140 x 120 mm, 23 parts, among them J1 Conn_02x20_Odd_Even, J2 Conn_02x02_Odd_Even, J3 Conn_02x02_Odd_Even, J4 Conn_02x04_Odd_Even

Commit message: Properly filled document metadata
Other:
- board text removed: "RSHP-CB-0010"
Changed lines of the file:
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@@
   )
   (paper "A4")
+  (title_block
+    (title "RSHP-CB-0010")
+    (date "2022-05-21")
+    (rev "1.0")
+    (company "(c) Andriy Golovnya http://redscorp.net")
+    (comment 1 "Reflow Soldering Hot Plate - Connection Board")
+  )
   (layers
     (0 "F.Cu" signal)
@@
     (effects (font (size 1.5 1.5) (thickness 0.3)))
   )
-  (gr_text "RSHP-CB-0010" (at 187.5 190) (layer "User.1")
-    (effects (font (size 1 1) (thickness 0.15)) (justify left))
-  )
   (via (at 52.5 110) (size 0.8) (drill 0.4) (layers "F.Cu" "B.Cu") (free) (net 3))
